Commit message: Add files via upload

File: track_bot_sim/urdf/gazebo.xacro (robot description, xacro)
@@ -1,19 +1,35 @@
 <?xml version="1.0"?>
 <robot xmlns:xacro="http://www.ros.org/wiki/xacro" name="track_bot">
+<!-- ***** Wheel Setup ***** -->
+    <xacro:macro name="wheel_setup">
+        <material>Gazebo/Blue</material>
+        <mu1>1</mu1>
+        <mu2>1</mu2>
+        <!-- <slip1>0.0</slip1>
+        <slip2>0.0</slip2>
+        <kp>1e6</kp>
+        <kd>1.0</kd>
+        <maxVel>0.1</maxVel>
+        <minDepth>0.001</minDepth> -->
+    </xacro:macro>
+<!-- ***** Wheel Setup End***** -->
+<!-- ***** Gazebo Setup ***** -->
     <gazebo reference="body_link">
         <material>Gazebo/Green</material>
     </gazebo>
     <gazebo reference="FR_wheel_link">
-        <material>Gazebo/Blue</material>
+        <xacro:wheel_setup/>
     </gazebo>
     <gazebo reference="FL_wheel_link">
-        <material>Gazebo/Blue</material>
+        <xacro:wheel_setup/>
     </gazebo>
     <gazebo reference="RR_wheel_link">
-        <material>Gazebo/Blue</material>
+        <xacro:wheel_setup/>
     </gazebo>
     <gazebo reference="RL_wheel_link">
-        <material>Gazebo/Blue</material>
+        <xacro:wheel_setup/>
     </gazebo>
+<!-- ***** Gazebo Setup End ***** -->
+<!-- ***** Gazebo Plugins ***** -->
     <gazebo>
         <plugin name="gazebo_ros2_control" filename="libgazebo_ros2_control.so">
@@ -26,4 +42,6 @@
         </plugin>
     </gazebo>
+<!-- ***** Gazebo Plugins End***** -->
+<!-- ***** Gazebo Control ***** -->
     <ros2_control name="GazeboSystem" type="system">
     <hardware>
@@ -31,35 +49,64 @@
     </hardware>
     <joint name="FR_wheel_joint">
-        <command_interface name="velocity">
+        <!-- <command_interface name="velocity">
+            <param name="max">10</param>
             <param name="min">-10</param>
-            <param name="max">10</param>
-        </command_interface>
+        </command_interface> -->
         <state_interface name="velocity"/>
         <state_interface name="position"/>
+        <command_interface name="velocity"/>
     </joint>
     <joint name="FL_wheel_joint">
-        <command_interface name="velocity">
-            <param name="min">-10</param>
-            <param name="max">10</param>
-        </command_interface>
         <state_interface name="velocity"/>
         <state_interface name="position"/>
+        <command_interface name="velocity"/>
     </joint>
     <joint name="RR_wheel_joint">
-        <command_interface name="velocity">
-            <param name="min">-10</param>
-            <param name="max">10</param>
-        </command_interface>
         <state_interface name="velocity"/>
         <state_interface name="position"/>
+        <command_interface name="velocity"/>
     </joint>
     <joint name="RL_wheel_joint">
-        <command_interface name="velocity">
-            <param name="min">-10</param>
-            <param name="max">10</param>
-        </command_interface>
         <state_interface name="velocity"/>
         <state_interface name="position"/>
+        <command_interface name="velocity"/>
     </joint>
     </ros2_control>
+<!-- ***** Gazebo Control End ***** -->
+<!-- ***** Camera Parts ***** -->
+    <joint name="camera_optical_joint" type="fixed">
+        <origin xyz="0 0 0" rpy="-1.571 0 -1.571" />
+        <parent link="camera_link" />
+        <child link="camera_link_optical" />
+    </joint>
+    <link name="camera_link_optical"></link>
+    <gazebo reference="camera_link">
+        <sensor type="depth" name="my_camera">
+            <update_rate>20</update_rate>
+            <visualize>true</visualize>
+            <camera name="cam">
+                <horizontal_fov>1.3962634</horizontal_fov>
+                <image>
+                    <width>640</width>
+                    <height>480</height>
+                    <format>R8B8G8</format>
+                </image>
+                <clip>
+                    <near>0.02</near>
+                    <far>300</far>
+                </clip>
+                <noise>
+                    <type>gaussian</type>
+                    <mean>0.0</mean>
+                    <stddev>0.007</stddev>
+                </noise>
+            </camera>
+            <plugin name="camera_controller" filename="libgazebo_ros_camera.so">
+                <frame_name>camera_link_optical</frame_name>
+                <min_depth>0.1</min_depth>
+                <max_depth>500</max_depth>
+            </plugin>
+        </sensor>
+    </gazebo>
+<!-- ***** Camera Parts End ***** -->
 </robot>

File: track_bot_sim/urdf/model.urdf.xacro (robot description, xacro)
@@ -33,5 +33,5 @@
         </xacro:inertial_box>
     </xacro:macro>
-<!-- ***** Body Setup End***** -->
+<!-- ***** Body Setup End ***** -->
 <!-- ***** Wheel Setup ***** -->
     <xacro:property name="wheel_origin_x" value="0.8"/>
@@ -40,5 +40,5 @@
     <xacro:property name="wheel_radius" value="0.5"/>
     <xacro:property name="wheel_length" value="0.25"/>
-    <xacro:property name="wheel_mass" value="0.25"/>
+    <xacro:property name="wheel_mass" value="5"/>
     <xacro:macro name="wheel_shape">
         <geometry>
@@ -66,4 +66,5 @@
 <!-- ***** Wheel Setup End ***** -->
     <link name="base_link"></link>
+<!-- ***** Body Parts ***** -->
     <joint name="body_joint" type="fixed">
         <xacro:body_origin/>
@@ -74,4 +75,6 @@
         <xacro:body_link/>
     </link>
+<!-- ***** Body Parts End ***** -->
+<!-- ***** Wheel Parts ***** -->
     <joint name="FR_wheel_joint" type="continuous">
         <parent link="body_link"/>
@@ -110,4 +113,37 @@
         <xacro:wheel_link/>
     </link>
+<!-- ***** Wheel Parts End ***** -->
+<!-- ***** Camera Parts ***** -->
+    <joint name="camera_joint" type="fixed">
+        <origin xyz="0 0 2" rpy="0 0 0"/>
+        <parent link="body_link"/>
+        <child link="camera_link"/>
+    </joint>
+    <link name="camera_link">
+        <visual>
+            <origin xyz="-0.03 0 0" rpy="0 0 0"/>
+            <geometry>
+                <box size="0.06 0.15 0.15" />
+            </geometry>
+            <material name="white" />
+        </visual>
+        <visual>
+            <origin xyz="0.03 0 0" rpy="0 ${pi/2} 0"/>
+            <geometry>
+                <cylinder length="0.06" radius="0.04" />
+            </geometry>
+            <material name="blue" />
+        </visual>
+        <collision>
+            <origin xyz="0.0 0 0" rpy="0 0 0"/>
+            <geometry>
+                <box size="0.12 0.15 0.15" />
+            </geometry>
+        </collision>
+        <xacro:inertial_box mass="0.1" x="0.12" y="0.15" z="0.15">
+            <origin xyz="0.0 0 0" rpy="0 0 0"/>
+        </xacro:inertial_box>
+    </link>
+<!-- ***** Camera Parts End***** -->
     <xacro:include filename="gazebo.xacro"/>
 </robot>

Commit message: Add files via upload

File: track_bot_sim/urdf/gazebo.xacro (robot description, xacro)
@@ -110,3 +110,54 @@
     </gazebo>
 <!-- ***** Camera Parts End ***** -->
+<!-- ***** Lidar Parts ***** -->
+    <joint name="laser_joint" type="fixed">
+        <parent link="body_link"/>
+        <child link="laser_frame"/>
+        <origin xyz="0 0 1" rpy="0 0 0"/>
+    </joint>
+    <link name="laser_frame">
+        <visual>
+            <geometry>
+                <cylinder radius="0.05" length="0.04"/>
+            </geometry>
+            <material name="red"/>
+        </visual>
+        <collision>
+            <geometry>
+                <cylinder radius="0.05" length="0.04"/>
+            </geometry>
+        </collision>
+        <xacro:inertial_cylinder mass="0.1" length="0.04" radius="0.05">
+            <origin xyz="0 0 0" rpy="0 0 0"/>
+        </xacro:inertial_cylinder>
+    </link>
+    <gazebo reference="laser_frame">
+        <material>Gazebo/Red</material>
+        <sensor name="laser" type="ray">
+            <pose> 0 0 0 0 0 0 </pose>
+            <visualize>true</visualize>
+            <update_rate>10</update_rate>
+            <ray>
+                <scan>
+                    <horizontal>
+                        <samples>360</samples>
+                        <min_angle>-3.14</min_angle>
+                        <max_angle>3.14</max_angle>
+                    </horizontal>
+                </scan>
+                <range>
+                    <min>0.3</min>
+                    <max>12</max>
+                </range>
+            </ray>
+            <plugin name="laser_controller" filename="libgazebo_ros_ray_sensor.so">
+                <ros>
+                    <argument>~/out:=scan</argument>
+                </ros>
+                <output_type>sensor_msgs/LaserScan</output_type>
+                <frame_name>laser_frame</frame_name>
+            </plugin>
+        </sensor>
+    </gazebo>
+<!-- ***** Lidar Parts End***** -->
 </robot>

File: track_bot_sim/urdf/model.urdf.xacro (robot description, xacro)
@@ -36,8 +36,8 @@
 <!-- ***** Wheel Setup ***** -->
     <xacro:property name="wheel_origin_x" value="0.8"/>
-    <xacro:property name="wheel_origin_y" value="0.625"/>
-    <xacro:property name="wheel_origin_z" value="0"/>
-    <xacro:property name="wheel_radius" value="0.5"/>
-    <xacro:property name="wheel_length" value="0.25"/>
+    <xacro:property name="wheel_origin_y" value="0.75"/>
+    <xacro:property name="wheel_origin_z" value="-0.5"/>
+    <xacro:property name="wheel_radius" value="0.25"/>
+    <xacro:property name="wheel_length" value="0.5"/>
     <xacro:property name="wheel_mass" value="5"/>
     <xacro:macro name="wheel_shape">
@@ -80,5 +80,5 @@
         <parent link="body_link"/>
         <child link="FR_wheel_link"/>
-        <origin xyz="${wheel_origin_x} -${wheel_origin_y} ${wheel_origin_z}" rpy="-${pi/2} 0 0"/>
+        <origin xyz="${wheel_origin_x} -${wheel_origin_y} ${wheel_origin_z}" rpy="${pi/2} 0 0"/>
         <xacro:wheel_axis/>
     </joint>
@@ -98,5 +98,5 @@
         <parent link="body_link"/>
         <child link="RR_wheel_link"/>
-        <origin xyz="-${wheel_origin_x} -${wheel_origin_y} ${wheel_origin_z}" rpy="-${pi/2} 0 0"/>
+        <origin xyz="-${wheel_origin_x} -${wheel_origin_y} ${wheel_origin_z}" rpy="${pi/2} 0 0"/>
         <xacro:wheel_axis/>
     </joint>
