Commit message: Add files via upload

File: track_bot_sim/urdf/gazebo.xacro (robot description, xacro)
@@ -1,34 +1,63 @@
 <?xml version="1.0"?>
-<robot xmlns:xacro="http://www.ros.org/wiki/xacro" name="track_bot">
-<!-- ***** Wheel Setup ***** -->
-    <xacro:macro name="wheel_setup">
-        <material>Gazebo/Blue</material>
-        <mu1>1</mu1>
-        <mu2>1</mu2>
-        <!-- <slip1>0.0</slip1>
-        <slip2>0.0</slip2>
-        <kp>1e6</kp>
-        <kd>1.0</kd>
-        <maxVel>0.1</maxVel>
-        <minDepth>0.001</minDepth> -->
-    </xacro:macro>
-<!-- ***** Wheel Setup End***** -->
-<!-- ***** Gazebo Setup ***** -->
-    <gazebo reference="body_link">
-        <material>Gazebo/Green</material>
+<robot xmlns:xacro="http://www.ros.org/wiki/xacro">
+<!-- ***** Camera Plugin ***** -->
+    <gazebo reference="camera_sensor_link">
+        <sensor type="depth" name="camera_sensor">
+            <update_rate>20</update_rate>
+            <visualize>true</visualize>
+            <camera name="cam">
+                <horizontal_fov>1.3962634</horizontal_fov>
+                <image>
+                    <width>640</width>
+                    <height>480</height>
+                    <format>R8B8G8</format>
+                </image>
+                <clip>
+                    <near>0.02</near>
+                    <far>300</far>
+                </clip>
+                <noise>
+                    <type>gaussian</type>
+                    <mean>0.0</mean>
+                    <stddev>0.007</stddev>
+                </noise>
+            </camera>
+            <plugin name="camera_controller" filename="libgazebo_ros_camera.so">
+                <frame_name>camera_optical_link</frame_name>
+                <min_depth>0.1</min_depth>
+                <max_depth>500</max_depth>
+            </plugin>
+        </sensor>
     </gazebo>
-    <gazebo reference="FR_wheel_link">
-        <xacro:wheel_setup/>
+<!-- ***** Camera Plugin End ***** -->
+<!-- ***** Lidar Plugin ***** -->
+    <gazebo reference="lidar_sensor_link">
+        <sensor name="laser" type="ray">
+            <pose> 0 0 0 0 0 0 </pose>
+            <visualize>true</visualize>
+            <update_rate>10</update_rate>
+            <ray>
+                <scan>
+                    <horizontal>
+                        <samples>360</samples>
+                        <min_angle>-3.14</min_angle>
+                        <max_angle>3.14</max_angle>
+                    </horizontal>
+                </scan>
+                <range>
+                    <min>0.3</min>
+                    <max>12</max>
+                </range>
+            </ray>
+            <plugin name="laser_controller" filename="libgazebo_ros_ray_sensor.so">
+                <ros>
+                    <argument>~/out:=scan</argument>
+                </ros>
+                <output_type>sensor_msgs/LaserScan</output_type>
+                <frame_name>lidar_sensor_link</frame_name>
+            </plugin>
+        </sensor>
     </gazebo>
-    <gazebo reference="FL_wheel_link">
-        <xacro:wheel_setup/>
-    </gazebo>
-    <gazebo reference="RR_wheel_link">
-        <xacro:wheel_setup/>
-    </gazebo>
-    <gazebo reference="RL_wheel_link">
-        <xacro:wheel_setup/>
-    </gazebo>
-<!-- ***** Gazebo Setup End ***** -->
+<!-- ***** Lidar Plugin End ***** -->
 <!-- ***** Gazebo Plugins ***** -->
     <gazebo>
@@ -74,90 +103,45 @@
     </ros2_control>
 <!-- ***** Gazebo Control End ***** -->
-<!-- ***** Camera Parts ***** -->
-    <joint name="camera_optical_joint" type="fixed">
-        <origin xyz="0 0 0" rpy="-1.571 0 -1.571" />
-        <parent link="camera_link" />
-        <child link="camera_link_optical" />
-    </joint>
-    <link name="camera_link_optical"></link>
+<!-- ***** Wheel Setup ***** -->
+    <xacro:macro name="wheel_setup">
+        <material>Gazebo/Blue</material>
+        <mu1>1</mu1>
+        <mu2>1</mu2>
+        <!-- <slip1>0.0</slip1>
+        <slip2>0.0</slip2>
+        <kp>1e6</kp>
+        <kd>1.0</kd>
+        <maxVel>0.1</maxVel>
+        <minDepth>0.001</minDepth> -->
+    </xacro:macro>
+<!-- ***** Wheel Setup End***** -->
+<!-- ***** Gazebo Setup ***** -->
+    <gazebo reference="body_link">
+        <material>Gazebo/Green</material>
+    </gazebo>
+    <gazebo reference="FR_wheel_link">
+        <xacro:wheel_setup/>
+    </gazebo>
+    <gazebo reference="FL_wheel_link">
+        <xacro:wheel_setup/>
+    </gazebo>
+    <gazebo reference="RR_wheel_link">
+        <xacro:wheel_setup/>
+    </gazebo>
+    <gazebo reference="RL_wheel_link">
+        <xacro:wheel_setup/>
+    </gazebo>
     <gazebo reference="camera_link">
-        <sensor type="depth" name="my_camera">
-            <update_rate>20</update_rate>
-            <visualize>true</visualize>
-            <camera name="cam">
-                <horizontal_fov>1.3962634</horizontal_fov>
-                <image>
-                    <width>640</width>
-                    <height>480</height>
-                    <format>R8B8G8</format>
-                </image>
-                <clip>
-                    <near>0.02</near>
-                    <far>300</far>
-                </clip>
-                <noise>
-                    <type>gaussian</type>
-                    <mean>0.0</mean>
-                    <stddev>0.007</stddev>
-                </noise>
-            </camera>
-            <plugin name="camera_controller" filename="libgazebo_ros_camera.so">
-                <frame_name>camera_link_optical</frame_name>
-                <min_depth>0.1</min_depth>
-                <max_depth>500</max_depth>
-            </plugin>
-        </sensor>
+        <material>Gazebo/Red</material>
     </gazebo>
-<!-- ***** Camera Parts End ***** -->
-<!-- ***** Lidar Parts ***** -->
-    <joint name="laser_joint" type="fixed">
-        <parent link="body_link"/>
-        <child link="laser_frame"/>
-        <origin xyz="0 0 1" rpy="0 0 0"/>
-    </joint>
-    <link name="laser_frame">
-        <visual>
-            <geometry>
-                <cylinder radius="0.05" length="0.04"/>
-            </geometry>
-            <material name="red"/>
-        </visual>
-        <collision>
-            <geometry>
-                <cylinder radius="0.05" length="0.04"/>
-            </geometry>
-        </collision>
-        <xacro:inertial_cylinder mass="0.1" length="0.04" radius="0.05">
-            <origin xyz="0 0 0" rpy="0 0 0"/>
-        </xacro:inertial_cylinder>
-    </link>
-    <gazebo reference="laser_frame">
+    <gazebo reference="camera_sensor_link">
         <material>Gazebo/Red</material>
-        <sensor name="laser" type="ray">
-            <pose> 0 0 0 0 0 0 </pose>
-            <visualize>true</visualize>
-            <update_rate>10</update_rate>
-            <ray>
-                <scan>
-                    <horizontal>
-                        <samples>360</samples>
-                        <min_angle>-3.14</min_angle>
-                        <max_angle>3.14</max_angle>
-                    </horizontal>
-                </scan>
-                <range>
-                    <min>0.3</min>
-                    <max>12</max>
-                </range>
-            </ray>
-            <plugin name="laser_controller" filename="libgazebo_ros_ray_sensor.so">
-                <ros>
-                    <argument>~/out:=scan</argument>
-                </ros>
-                <output_type>sensor_msgs/LaserScan</output_type>
-                <frame_name>laser_frame</frame_name>
-            </plugin>
-        </sensor>
     </gazebo>
-<!-- ***** Lidar Parts End***** -->
+    <gazebo reference="lidar_link">
+        <material>Gazebo/Red</material>
+    </gazebo>
+    <gazebo reference="lidar_sensor_link">
+        <material>Gazebo/Red</material>
+    </gazebo>
+<!-- ***** Gazebo Setup End ***** -->
 </robot>

File: track_bot_sim/urdf/model.urdf.xacro (robot description, xacro)
@@ -1,5 +1,5 @@
 <?xml version="1.0"?>
 <robot xmlns:xacro="http://www.ros.org/wiki/xacro" name="track_bot">
-    <xacro:include filename="setup.xacro"/>
+    <xacro:include filename="funtions.xacro"/>
 <!-- ***** Body Setup ***** -->
     <xacro:property name="body_origin_x" value="0"/>
@@ -9,5 +9,5 @@
     <xacro:property name="body_size_y" value="1"/>
     <xacro:property name="body_size_z" value="0.5"/>
-    <xacro:property name="body_mass" value="1"/>
+    <xacro:property name="body_mass" value="10"/>
     <xacro:macro name="body_origin">
         <origin xyz="${body_origin_x} ${body_origin_y} ${body_origin_z}" rpy="0 0 0"/>
@@ -30,5 +30,5 @@
         </collision>
         <xacro:inertial_box mass="${body_mass}" x="${body_size_x}" y="${body_size_y}" z="${body_size_z}">
-            <xacro:body_origin/>
+            <origin xyz="0 0 0" rpy="0 0 0"/>
         </xacro:inertial_box>
     </xacro:macro>
@@ -41,5 +41,9 @@
     <xacro:property name="wheel_length" value="0.5"/>
     <xacro:property name="wheel_mass" value="5"/>
+    <xacro:macro name="wheel_offset_origin">
+        <origin xyz="0 0 ${wheel_length/2}" rpy="0 0 0"/>
+    </xacro:macro>
     <xacro:macro name="wheel_shape">
+        <xacro:wheel_offset_origin/>
         <geometry>
             <cylinder radius="${wheel_radius}" length="${wheel_length}"/>
@@ -61,8 +65,77 @@
         </collision>
         <xacro:inertial_cylinder mass="${wheel_mass}" length="${wheel_length}" radius="${wheel_radius}">
-            <origin xyz="0 0 0" rpy="0 0 0"/>
+            <xacro:wheel_offset_origin/>
         </xacro:inertial_cylinder>
     </xacro:macro>
 <!-- ***** Wheel Setup End ***** -->
+<!-- ***** Camera Setup ***** -->
+    <xacro:property name="camera_origin_x" value="1"/>
+    <xacro:property name="camera_origin_y" value="0"/>
+    <xacro:property name="camera_origin_z" value="0.5"/>
+    <xacro:property name="camera_size_x" value="0.1"/>
+    <xacro:property name="camera_size_y" value="0.2"/>
+    <xacro:property name="camera_size_z" value="0.2"/>
+    <xacro:property name="camera_sensor_length" value="0.05"/>
+    <xacro:property name="camera_sensor_radius" value="0.05"/>
+    <xacro:property name="camera_mass" value="0.001"/>
+    <xacro:macro name="camera_origin">
+        <origin xyz="${camera_origin_x} ${camera_origin_y} ${camera_origin_z}" rpy="0 0 0"/>
+    </xacro:macro>
+    <xacro:macro name="camera_offset_origin">
+        <origin xyz="${camera_size_x/2} 0 0" rpy="0 0 0"/>
+    </xacro:macro>
+    <xacro:macro name="camera_sensor_offset_origin">
+        <origin xyz="${camera_sensor_length/2} 0 0" rpy="0 ${pi/2} 0"/>
+    </xacro:macro>
+    <xacro:macro name="camera_shape">
+        <xacro:camera_offset_origin/>
+        <geometry>
+            <box size="${camera_size_x} ${camera_size_y} ${camera_size_z}"/>
+        </geometry>
+    </xacro:macro>
+    <xacro:macro name="camera_sensor_shape">
+        <xacro:camera_sensor_offset_origin/>
+        <geometry>
+            <cylinder length="${camera_sensor_length}" radius="${camera_sensor_radius}"/>
+        </geometry>
+    </xacro:macro>
+    <xacro:macro name="camera_color">
+        <material name="red"/>
+    </xacro:macro>
+<!-- ***** Camera Setup End***** -->
+<!-- ***** Lidar Setup ***** -->
+    <xacro:property name="lidar_origin_x" value="0"/>
+    <xacro:property name="lidar_origin_y" value="0"/>
+    <xacro:property name="lidar_origin_z" value="0.75"/>
+    <xacro:property name="lidar_radius" value="0.1"/>
+    <xacro:property name="lidar_length" value="0.1"/>
+    <xacro:property name="lidar_sensor_radius" value="0.08"/>
+    <xacro:property name="lidar_sensor_length" value="0.08"/>
+    <xacro:property name="lidar_mass" value="0.001"/>
+    <xacro:macro name="lidar_origin">
+        <origin xyz="${lidar_origin_x} ${lidar_origin_y} ${lidar_origin_z}" rpy="0 0 0"/>
+    </xacro:macro>
+    <xacro:macro name="lidar_offset_origin">
+        <origin xyz="0 0 ${lidar_length/2}" rpy="0 0 0"/>
+    </xacro:macro>
+    <xacro:macro name="lidar_sensor_offset_origin">
+        <origin xyz="0 0 ${lidar_sensor_length/2}" rpy="0 0 0"/>
+    </xacro:macro>
+    <xacro:macro name="lidar_shape">
+        <xacro:lidar_offset_origin/>
+        <geometry>
+            <cylinder radius="${lidar_radius}" length="${lidar_length}"/>
+        </geometry>
+    </xacro:macro>
+    <xacro:macro name="lidar_sensor_shape">
+        <xacro:lidar_sensor_offset_origin/>
+        <geometry>
+            <cylinder length="${lidar_sensor_length}" radius="${lidar_sensor_radius}"/>
+        </geometry>
+    </xacro:macro>
+    <xacro:macro name="lidar_color">
+        <material name="red"/>
+    </xacro:macro>
+<!-- ***** Lidar Setup End ***** -->
     <link name="base_link"></link>
 <!-- ***** Body Parts ***** -->
@@ -116,5 +189,5 @@
 <!-- ***** Camera Parts ***** -->
     <joint name="camera_joint" type="fixed">
-        <origin xyz="0 0 2" rpy="0 0 0"/>
+        <xacro:camera_origin/>
         <parent link="body_link"/>
         <child link="camera_link"/>
@@ -122,28 +195,74 @@
     <link name="camera_link">
         <visual>
-            <origin xyz="-0.03 0 0" rpy="0 0 0"/>
-            <geometry>
-                <box size="0.06 0.15 0.15" />
-            </geometry>
-            <material name="white" />
-        </visual>
-        <visual>
-            <origin xyz="0.03 0 0" rpy="0 ${pi/2} 0"/>
-            <geometry>
-                <cylinder length="0.06" radius="0.04" />
-            </geometry>
-            <material name="blue" />
-        </visual>
-        <collision>
-            <origin xyz="0.0 0 0" rpy="0 0 0"/>
-            <geometry>
-                <box size="0.12 0.15 0.15" />
-            </geometry>
-        </collision>
-        <xacro:inertial_box mass="0.1" x="0.12" y="0.15" z="0.15">
-            <origin xyz="0.0 0 0" rpy="0 0 0"/>
+            <xacro:camera_shape/>
+            <xacro:camera_color/>
+        </visual>
+        <collision>
+            <xacro:camera_shape/>
+        </collision>
+        <xacro:inertial_box mass="${camera_mass}" x="${camera_size_x}" y="${camera_size_y}" z="${camera_size_z}">
+            <xacro:camera_offset_origin/>
         </xacro:inertial_box>
     </link>
-<!-- ***** Camera Parts End***** -->
+    <joint name="camera_sensor_joint" type="fixed">
+        <origin xyz="${camera_size_x} 0 0" rpy="0 0 0"/>
+        <parent link="camera_link"/>
+        <child link="camera_sensor_link"/>
+    </joint>
+    <link name="camera_sensor_link">
+        <visual>
+            <xacro:camera_sensor_shape/>
+            <xacro:camera_color/>
+        </visual>
+        <collision>
+            <xacro:camera_sensor_shape/>
+        </collision>
+        <xacro:inertial_cylinder mass="${camera_mass}" length="${camera_sensor_length}" radius="${camera_sensor_radius}">
+            <xacro:camera_sensor_offset_origin/>
+        </xacro:inertial_cylinder>
+    </link>
+    <joint name="camera_optical_joint" type="fixed">
+        <origin xyz="0 0 0" rpy="-${pi/2} 0 -${pi/2}"/>
+        <parent link="camera_sensor_link"/>
+        <child link="camera_optical_link"/>
+    </joint>
+    <link name="camera_optical_link"></link>
+<!-- ***** Camera Parts End ***** -->
+<!-- ***** Lidar Parts ***** -->
+    <joint name="lidar_joint" type="fixed">
+        <parent link="body_link"/>
+        <child link="lidar_link"/>
+        <xacro:lidar_origin/>
+    </joint>
+    <link name="lidar_link">
+        <visual>
+            <xacro:lidar_shape/>
+            <xacro:lidar_color/>
+        </visual>
+        <collision>
+            <xacro:lidar_shape/>
+        </collision>
+        <xacro:inertial_cylinder mass="${lidar_mass}" length="${lidar_length}" radius="${lidar_radius}">
+            <xacro:lidar_offset_origin/>
+        </xacro:inertial_cylinder>
+    </link>
+    <joint name="lidar_sensor_joint" type="fixed">
+        <origin xyz="0 0 ${lidar_length}" rpy="0 0 0"/>
+        <parent link="lidar_link"/>
+        <child link="lidar_sensor_link"/>
+    </joint>
+    <link name="lidar_sensor_link">
+        <visual>
+            <xacro:lidar_sensor_shape/>
+            <xacro:lidar_color/>
+        </visual>
+        <collision>
+            <xacro:lidar_sensor_shape/>
+        </collision>
+        <xacro:inertial_cylinder mass="${lidar_mass}" length="${lidar_sensor_length}" radius="${lidar_sensor_radius}">
+            <xacro:lidar_sensor_offset_origin/>
+        </xacro:inertial_cylinder>
+    </link>
+<!-- ***** Lidar Parts End ***** -->
     <xacro:include filename="gazebo.xacro"/>
 </robot>
