Commit message: Add files via upload

File: track_bot_sim/urdf/gazebo.xacro (robot description, xacro)
@@ -17,11 +17,11 @@
                     <far>300</far>
                 </clip>
-                <noise>
+                <!-- <noise>
                     <type>gaussian</type>
                     <mean>0.0</mean>
                     <stddev>0.007</stddev>
-                </noise>
+                </noise> -->
             </camera>
-            <plugin name="camera_controller" filename="libgazebo_ros_camera.so">
+            <plugin name="camera_sensor" filename="libgazebo_ros_camera.so">
                 <frame_name>camera_optical_link</frame_name>
                 <min_depth>0.1</min_depth>
@@ -41,6 +41,6 @@
                     <horizontal>
                         <samples>360</samples>
-                        <min_angle>-3.14</min_angle>
-                        <max_angle>3.14</max_angle>
+                        <min_angle>-${pi}</min_angle>
+                        <max_angle>${pi}</max_angle>
                     </horizontal>
                 </scan>
@@ -49,6 +49,11 @@
                     <max>12</max>
                 </range>
+                <!-- <noise>
+                    <type>gaussian</type>
+                    <mean>0.0</mean>
+                    <stddev>0.01</stddev>
+                </noise> -->
             </ray>
-            <plugin name="laser_controller" filename="libgazebo_ros_ray_sensor.so">
+            <plugin name="lidar_sensor" filename="libgazebo_ros_ray_sensor.so">
                 <ros>
                     <argument>~/out:=scan</argument>
@@ -60,4 +65,45 @@
     </gazebo>
 <!-- ***** Lidar Plugin End ***** -->
+<!-- ***** Ultrasoni Sensor Plugin ***** -->
+    <gazebo reference="ultrasonic_link">
+        <sensor name="ultrasonic" type="ray">
+            <pose> 0 0 0 0 0 0 </pose>
+            <visualize>true</visualize>
+            <update_rate>10</update_rate>
+            <ray>
+                <scan>
+                    <horizontal>
+                        <samples>5</samples>
+                        <resolution>1.000000</resolution>
+                        <min_angle>-0.12</min_angle>
+                        <max_angle>0.12</max_angle>
+                    </horizontal>
+                    <vertical>
+                        <samples>5</samples>
+                        <resolution>1.000000</resolution>
+                        <min_angle>-0.01</min_angle>
+                        <max_angle>0.01</max_angle>
+                    </vertical>
+                </scan>
+                <range>
+                    <min>0.01</min>
+                    <max>4</max>
+                </range>
+                <!-- <noise>
+                    <type>gaussian</type>
+                    <mean>0.0</mean>
+                    <stddev>0.01</stddev>
+                </noise> -->
+            </ray>
+            <plugin name="ultrasonic_sensor" filename="libgazebo_ros_ray_sensor.so">
+                <ros>
+                    <argument>~/out:=ultrasonic_sensor</argument>
+                </ros>
+                <output_type>sensor_msgs/LaserScan</output_type>
+                <frame_name>ultrasonic_link</frame_name>
+            </plugin>
+        </sensor>
+    </gazebo>
+<!-- ***** Ultrasoni Sensor Plugin End ***** -->
 <!-- ***** Gazebo Plugins ***** -->
     <gazebo>
@@ -78,26 +124,34 @@
     </hardware>
     <joint name="FR_wheel_joint">
-        <!-- <command_interface name="velocity">
-            <param name="max">10</param>
-            <param name="min">-10</param>
-        </command_interface> -->
-        <state_interface name="velocity"/>
-        <state_interface name="position"/>
-        <command_interface name="velocity"/>
+        <state_interface name="velocity"/>
+        <state_interface name="position"/>
+        <command_interface name="velocity">
+            <param name="max">1</param>
+            <param name="min">-1</param>
+        </command_interface>
     </joint>
     <joint name="FL_wheel_joint">
         <state_interface name="velocity"/>
         <state_interface name="position"/>
-        <command_interface name="velocity"/>
+        <command_interface name="velocity">
+            <param name="max">1</param>
+            <param name="min">-1</param>
+        </command_interface>
     </joint>
     <joint name="RR_wheel_joint">
         <state_interface name="velocity"/>
         <state_interface name="position"/>
-        <command_interface name="velocity"/>
+        <command_interface name="velocity">
+            <param name="max">1</param>
+            <param name="min">-1</param>
+        </command_interface>
     </joint>
     <joint name="RL_wheel_joint">
         <state_interface name="velocity"/>
         <state_interface name="position"/>
-        <command_interface name="velocity"/>
+        <command_interface name="velocity">
+            <param name="max">1</param>
+            <param name="min">-1</param>
+        </command_interface>
     </joint>
     </ros2_control>
@@ -110,5 +164,5 @@
         <!-- <slip1>0.0</slip1>
         <slip2>0.0</slip2>
-        <kp>1e6</kp>
+        <kp>10000000.0</kp>
         <kd>1.0</kd>
         <maxVel>0.1</maxVel>

File: track_bot_sim/urdf/model.urdf.xacro (robot description, xacro)
@@ -36,5 +36,5 @@
 <!-- ***** Wheel Setup ***** -->
     <xacro:property name="wheel_origin_x" value="0.8"/>
-    <xacro:property name="wheel_origin_y" value="0.75"/>
+    <xacro:property name="wheel_origin_y" value="0.5"/>
     <xacro:property name="wheel_origin_z" value="-0.5"/>
     <xacro:property name="wheel_radius" value="0.25"/>
@@ -154,5 +154,6 @@
         <child link="FR_wheel_link"/>
         <origin xyz="${wheel_origin_x} -${wheel_origin_y} ${wheel_origin_z}" rpy="${pi/2} 0 0"/>
-        <xacro:wheel_axis/>
+        <axis xyz="0 0 -1"/>
+        <dynamics damping="1.0" friction="1.0"/>
     </joint>
     <link name="FR_wheel_link">
@@ -163,5 +164,6 @@
         <child link="FL_wheel_link"/>
         <origin xyz="${wheel_origin_x} ${wheel_origin_y} ${wheel_origin_z}" rpy="-${pi/2} 0 0"/>
-        <xacro:wheel_axis/>
+        <axis xyz="0 0 1"/>
+        <dynamics damping="1.0" friction="1.0"/>
     </joint>
     <link name="FL_wheel_link">
@@ -172,5 +174,6 @@
         <child link="RR_wheel_link"/>
         <origin xyz="-${wheel_origin_x} -${wheel_origin_y} ${wheel_origin_z}" rpy="${pi/2} 0 0"/>
-        <xacro:wheel_axis/>
+        <axis xyz="0 0 -1"/>
+        <dynamics damping="1.0" friction="1.0"/>
     </joint>
     <link name="RR_wheel_link">
@@ -181,5 +184,6 @@
         <child link="RL_wheel_link"/>
         <origin xyz="-${wheel_origin_x} ${wheel_origin_y} ${wheel_origin_z}" rpy="-${pi/2} 0 0"/>
-        <xacro:wheel_axis/>
+        <axis xyz="0 0 1"/>
+        <dynamics damping="1.0" friction="1.0"/>
     </joint>
     <link name="RL_wheel_link">
@@ -231,7 +235,7 @@
 <!-- ***** Lidar Parts ***** -->
     <joint name="lidar_joint" type="fixed">
+        <xacro:lidar_origin/>
         <parent link="body_link"/>
         <child link="lidar_link"/>
-        <xacro:lidar_origin/>
     </joint>
     <link name="lidar_link">
@@ -265,4 +269,18 @@
     </link>
 <!-- ***** Lidar Parts End ***** -->
+<!-- ***** Ultrasoni Sensor Parts ***** -->
+    <joint name="ultrasonic_joint" type="fixed">
+        <origin xyz="1.5 0 0" rpy="0 0 0"/>
+        <parent link="body_link"/>
+        <child link="ultrasonic_link"/>
+    </joint>
+    <link name="ultrasonic_link">
+        <visual>
+            <geometry>
+                <box size="0.05 0.2 0.1"/>
+            </geometry>
+        </visual>
+    </link>
+<!-- ***** Ultrasoni Sensor Parts End ***** -->
     <xacro:include filename="gazebo.xacro"/>
 </robot>
